File: pcb/glasses.brd (EAGLE design)
At the start: 158.8 x 54 mm, 93 parts, among them J2 JST-ZH-5SMD-RA, U1 WS2812, U10 WS2812, U11 WS2812, U12 WS2812, U13 WS2812, U14 WS2812, U15 WS2812, U16 WS2812, U17 WS2812, U18 WS2812, U19 WS2812, U2 WS2812, U20 WS2812, U21 WS2812, U22 WS2812, U23 WS2812, U24 WS2812, U25 WS2812, U26 WS2812, U27 WS2812, U28 WS2812, U29 WS2812, U3 WS2812, U30 WS2812, U31 WS2812, U32 WS2812, U33 WS2812, U34 WS2812, U35 WS2812, U36 WS2812, U37 WS2812, U38 WS2812, U39 WS2812, U4 WS2812, U40 WS2812, U41 WS2812, U42 WS2812, U43 WS2812, U44 WS2812, U45 WS2812, U46 WS2812, U47 WS2812, U48 WS2812, U49 WS2812, U5 WS2812, U50 WS2812, U51 WS2812, U52 WS2812, U53 WS2812, U54 WS2812, U55 WS2812, U56 WS2812, U57 WS2812, U58 WS2812, U59 WS2812, U6 WS2812, U60 WS2812, U61 32U4, U7 WS2812, U8 WS2812, U9 WS2812, X1 ECS-160-20-3X-TR

Commit message: ran DRC and moved vias
Routing:
- net +5V: track 7.70 -> 6.39 mm
Changed lines of the file:
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@@
 <contactref element="J1" pad="VBUS"/>
 <wire x1="5.35" y1="47.55" x2="5.3" y2="47.5" width="0.127" layer="1" curve="-90"/>
-<wire x1="5.3" y1="47.5" x2="4.6875" y2="47.5" width="0.127" layer="1"/>
 <wire x1="5.35" y1="47.55" x2="5.675" y2="47.55" width="0.4064" layer="1"/>
 <wire x1="6.25" y1="48.125" x2="5.675" y2="47.55" width="0.4064" layer="1" curve="90"/>
-<wire x1="6.25" y1="48.125" x2="6.875" y2="48.125" width="0.508" layer="1"/>
 <wire x1="5.35" y1="47.55" x2="7.1375" y2="47.55" width="0.4064" layer="1"/>
-<wire x1="7.1375" y1="47.55" x2="7.1875" y2="47.5" width="0.508" layer="1" curve="-90"/>
 <contactref element="J2" pad="P$1"/>
 <via x="86.575" y="48.6375" extent="1-16" drill="0.35"/>
@@
 <wire x1="7.45" y1="44.95" x2="7.5" y2="45" width="0.4064" layer="1" curve="90"/>
 <via x="7.5" y="45" extent="1-16" drill="0.35"/>
-<wire x1="70.96145625" y1="35.96145625" x2="70.3125" y2="35.3125" width="0.254" layer="1"/>
-<via x="70.3125" y="35.3125" extent="1-16" drill="0.2"/>
-<wire x1="72.83645625" y1="34.08645625" x2="72.1875" y2="33.4375" width="0.254" layer="1"/>
-<via x="72.1875" y="33.4375" extent="1-16" drill="0.2"/>
+<wire x1="70.96145625" y1="35.96145625" x2="70.2125" y2="35.2125" width="0.254" layer="1"/>
+<via x="70.2125" y="35.2125" extent="1-16" drill="0.2"/>
+<wire x1="72.83645625" y1="34.08645625" x2="72.0875" y2="33.3375" width="0.254" layer="1"/>
+<via x="72.0875" y="33.3375" extent="1-16" drill="0.2"/>
 <wire x1="74.71145625" y1="47.476040625" x2="74.56485" y2="47.54090625" width="0.127" layer="1" curve="45"/>
 <wire x1="74.56485" y1="47.54090625" x2="73.94934375" y2="48.218159375" width="0.127" layer="1"/>
@@
 <contactref element="C19" pad="2"/>
 <contactref element="C18" pad="2"/>
-<wire x1="69.08645625" y1="37.83645625" x2="68.471103125" y2="37.221103125" width="0.1524" layer="1"/>
-<wire x1="68.471103125" y1="37.221103125" x2="68.450678125" y2="37.17179375" width="0.1524" layer="1" curve="45"/>
-<via x="68.450678125" y="37.17179375" extent="1-16" drill="0.2"/>
+<wire x1="69.08645625" y1="37.83645625" x2="68.371103125" y2="37.121103125" width="0.1524" layer="1"/>
+<wire x1="68.371103125" y1="37.121103125" x2="68.350678125" y2="37.07179375" width="0.1524" layer="1" curve="45"/>
+<via x="68.350678125" y="37.07179375" extent="1-16" drill="0.2"/>
 <via x="79.990821875" y="37.545025" extent="1-16" drill="0.2"/>
 <wire x1="153.6" y1="49.25" x2="155" y2="49.25" width="0.4064" layer="1"/>
@@
 <contactref element="C13" pad="1"/>
 <contactref element="U61" pad="6"/>
-<wire x1="75.913540625" y1="46.27395625" x2="75.84283125" y2="46.20324375" width="0.127" layer="1"/>
 <wire x1="75.913540625" y1="46.27395625" x2="76.95914375" y2="45.840853125" width="0.1524" layer="1" curve="-45"/>
 <wire x1="76.95914375" y1="45.840853125" x2="77.595834375" y2="45.2041625" width="0.1524" layer="1"/>
@@
 <wire x1="77.6625" y1="41.1375" x2="79.658578125" y2="39.141421875" width="0.1524" layer="16"/>
 <wire x1="80.341421875" y1="39.141421875" x2="83.685340625" y2="42.485340625" width="0.1524" layer="16"/>
-<wire x1="76.181621875" y1="41.81005" x2="75.992890625" y2="41.62131875" width="0.1524" layer="1"/>
 <wire x1="76.181621875" y1="41.81005" x2="75.510784375" y2="41.1392125" width="0.1524" layer="1"/>
 <wire x1="75.510784375" y1="41.1392125" x2="75.5125" y2="41.1375" width="0.1524" layer="1"/>
@@
 <mfgpreviewcolor name="substratecolor" color="0xFF786E46"/>
 </mfgpreviewcolors>
+<errors>
+</errors>
 </board>
 </drawing>
